File: Pins/Diagram.sch (EAGLE design)
At the start: 26 parts, among them M1 MOTOR37MM, M2 MOTOR37MM, M3 MOTOR37MM, M4 MOTOR37MM, M5 MOTOR20MM, M6 MOTOR20MM, U1 L298, U2 BUCKCONVERTER

Commit message: Update pin table and wiring diagram for color sensor change. SCL and SDA are on D20 and D21. Thus, wheel M1EN has been moved to D12.
Parts:
- removed D1: LED-RGB-CC, ElectricalDiagramLibrary:LED-RGB-CC
- removed U$7: ENCODER, ElectricalDiagramLibrary:ENCODER
Connections:
- removed net N$58: B1.47, D1.GRN
- removed net N$59: B1.49, D1.BLU
- removed net N$60: B1.51/MOSI, D1.RED
- new net LOWER-DRIVER-REMAP: B1.12, U$1.DIO2(M1EN)
- net 5V: no longer U$7.VIN
- net GND: no longer U$7.GND
- net N$15: now also B1.20(SDA); no longer B1.2, U$1.DIO2(M1EN)
- net N$39: now also B1.3; no longer B1.18(TX1)
- net N$40: now also B1.2; no longer B1.19(RX1)
- net N$41: now also B1.18(TX1); no longer B1.20(SDA)
- net N$42: now also B1.19(RX1); no longer B1.21(SCL)
- net N$43: now also B1.11; no longer B1.30, U$7.OUTB
- net N$44: now also B1.21(SCL); no longer B1.3, U$7.OUTA
- net N$57: no longer D1.C
Other:
- note added: "Color Sensor"
- note added: "IR Reciever"
- note removed: "Belt encoder"
- note removed: "RGB SENS CON'S TEMPORARY"
- moved on the sheet: B1, BT1, F1, JP1, M1, M2, M3, M4, M5, M6, S1, S2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
